File: hardware/zero_crossing_detector_surface_mount/zero_crossing_detector.sch (KiCad schematic (older format))
At the start: 81 parts, among them J1 Conn_01x02, J2 BOOT0, J3 Conn_02x14_Odd_Even, J4 USB_B_Micro, J5 PowerSelect, J6 K-Type, J7 BOOT1, Q1 2N3904, SW1 Reset, U1 EL357N(C)(TA)-G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

Commit message: Changed to 5v AC-DC module. Added transistor to drive SSR output. Updated LDO
Parts:
- removed C20: 22uF, Capacitor_SMD:C_0603_1608Metric, symbol Device:C
- removed C3: 10uF, Capacitor_SMD:C_0805_2012Metric, symbol Device:CP
- removed J5: PowerSelect, Connector_PinHeader_2.54mm:PinHeader_1x03_P2.54mm_Vertical, symbol Connector_Generic:Conn_01x03
- removed U3: AMS1117, Package_TO_SOT_SMD:SOT-223-3_TabPin2, symbol Regulator_Linear:AMS1117
- added C3: 10uF, Capacitor_SMD:C_0402_1005Metric, symbol Device:C
- added D10, D11: B5819W, Diode_SMD:D_SOD-123, symbol Device:D_ALT
- added D12, D9: 1N4148, Diode_SMD:D_SOD-123, symbol Device:D_ALT
- added Q2, Q3: 2N3904, Package_TO_SOT_SMD:SOT-23, symbol Device:Q_NPN_BEC
- added R33, R34: 1k, Resistor_SMD:R_0402_1005Metric, symbol Device:R
- added R35: 10k, Resistor_SMD:R_0402_1005Metric, symbol Device:R
- added U3: AP2112K-3.3, Package_TO_SOT_SMD:SOT-23-5, symbol Regulator_Linear:AP2112K-3.3
- C18: value 4.7uf -> 10uF; LCSC Part Number C23733 -> C15525; Part Number CL05A475MP5NRNC -> CL05A106MQ5NUNC
- C19: value 22uF -> 100nF; footprint Capacitor_SMD:C_0603_1608Metric -> Capacitor_SMD:C_0402_1005Metric; LCSC Part Number C59461 -> C1525; Part Number CL10A226MQ8NRNC -> CL05B104KO5NNNC
- J3: value Conn_02x14_Odd_Even -> Conn_02x15_Odd_Even; footprint Connector_PinHeader_2.54mm:PinHeader_2x14_P2.54mm_Vertical -> Connector_PinHeader_2.54mm:PinHeader_2x15_P2.54mm_Vertical; symbol Connector_Generic:Conn_02x14_Odd_Even -> Connector_Generic:Conn_02x15_Odd_Even
- PS1: value HLK-PM03 -> HLK-PM01; symbol Converter_ACDC:HLK-PM03 -> Converter_ACDC:HLK-PM01; LCSC Part Number C209904 -> C209903; Part Number HLK-PM03 -> HLK-PM01
- R25, R26: value 1 -> 100k; LCSC Part Number C25086 -> C25741; Part Number 0402WGF100KTCE -> 0402WGF1003TCE
Connections:
- net labels added: +5V, 5V_MAINS, 5V_USB, MISC, MISC_RAW, SSR_RAW
- net labels removed: 3.3V_MAINS, 3.3V_USB, VBUS
- wire segments 209 -> 235
- no-connect marks 27 -> 26
Other:
- note added: "3.3v LDO"
- note added: "Mains 5V AC-DC"
- note added: "Misc output"
- note added: "SSR/Relay output"
- note removed: "3.3V Selector"
- note removed: "Mains 3.3V AC-DC"
- note removed: "USB 3.3v LDO"
- moved on the sheet: C4, R15

Commit message: Added tiny 1x1mm RGB LED to pcb
Parts:
- added D13: LED_ARBG, Custom:SMLP34RGB, symbol custom:LED_ARBG
- added R36: 220, Resistor_SMD:R_0402_1005Metric, symbol Device:R
- added R37: 75, Resistor_SMD:R_0402_1005Metric, symbol Device:R
- added R38: 47, Resistor_SMD:R_0402_1005Metric, symbol Device:R
- R7: value 10k -> 33; LCSC Part Number C25744 -> C25105; Part Number 0402WGF1002TCE -> 0402WGF330JTCE
- R8: value 150 -> 220; LCSC Part Number C25082 -> C25091; Part Number 0402WGF1500TCE -> 0402WGF2200TCE
Connections:
- net GND: no longer R7.2, R8.2
- net USR_LED: now also R8.2; no longer D7.2 (A), R7.1
- net VCC: now also D7.2 (A), D13.1 (A)
- net R_LED: now reaches U2.20 (PA4)
- net R_LED: now also R7.2
- net B_LED: now reaches U2.21 (PA5)
- net B_LED: now also R37.2
- net G_LED: now reaches U2.22 (PA6)
- net G_LED: now also R38.2
- new net: D13.2 (RK), R36.1
- new net: D13.3 (GK), R37.1
- new net: D13.4 (BK), R38.1
- new net: R36.2, R7.1
- no-connect marks 26 -> 23
Other:
- moved on the sheet: D7
Changed lines of the file:
@@
 Sheet 1 1
 Title "Zero crossing SSR Controller"
-Date "2019-11-11"
+Date "2019-11-15"
 Rev "0.2"
 Comp ""
@@
 $EndComp
 $Comp
-L Device:R R8
-U 1 1 5DA5DADD
-P 4500 6850
-F 0 "R8" H 4570 6896 50  0000 L CNN
-F 1 "150" H 4570 6805 50  0000 L CNN
-F 2 "Resistor_SMD:R_0402_1005Metric" V 4430 6850 50  0001 C CNN
-F 3 "~" H 4500 6850 50  0001 C CNN
-F 4 "0402WGF1500TCE" H 4500 6850 50  0001 C CNN "Part Number"
-F 5 "C25082" H 4500 6850 50  0001 C CNN "LCSC Part Number"
-	1    4500 6850
-	1    0    0    -1
-$EndComp
-$Comp
-L power:GND #PWR0135
-U 1 1 5DA5DAE9
-P 4500 7000
-F 0 "#PWR0135" H 4500 6750 50  0001 C CNN
-F 1 "GND" H 4505 6827 50  0000 C CNN
-F 2 "" H 4500 7000 50  0001 C CNN
-F 3 "" H 4500 7000 50  0001 C CNN
-	1    4500 7000
-	1    0    0    -1
-$EndComp
-$Comp
 L Device:LED D7
 U 1 1 5DA5DAF1
-P 4500 6550
-F 0 "D7" V 4447 6628 50  0000 L CNN
-F 1 "USR_Red" V 4538 6628 50  0000 L CNN
-F 2 "LED_SMD:LED_0603_1608Metric" H 4500 6550 50  0001 C CNN
-F 3 "~" H 4500 6550 50  0001 C CNN
-F 4 "红灯 0603" V 4500 6550 50  0001 C CNN "Part Number"
-F 5 "C2286" V 4500 6550 50  0001 C CNN "LCSC Part Number"
-	1    4500 6550
-	0    -1   -1   0
-$EndComp
-Text Label 4400 6200 0    50   ~ 0
+P 7450 2000
+F 0 "D7" H 7400 1900 50  0000 L CNN
+F 1 "USR_Red" H 7250 2100 50  0000 L CNN
+F 2 "LED_SMD:LED_0603_1608Metric" H 7450 2000 50  0001 C CNN
+F 3 "~" H 7450 2000 50  0001 C CNN
+F 4 "红灯 0603" V 7450 2000 50  0001 C CNN "Part Number"
+F 5 "C2286" V 7450 2000 50  0001 C CNN "LCSC Part Number"
+	1    7450 2000
+	1    0    0    -1
+$EndComp
+Text Label 6800 2000 2    50   ~ 0
 USR_LED
-$Comp
-L power:GND #PWR0136
-U 1 1 5DA7C477
-P 4250 7000
-F 0 "#PWR0136" H 4250 6750 50  0001 C CNN
-F 1 "GND" H 4255 6827 50  0000 C CNN
-F 2 "" H 4250 7000 50  0001 C CNN
-F 3 "" H 4250 7000 50  0001 C CNN
-	1    4250 7000
-	1    0    0    -1
-$EndComp
-Wire Wire Line
-	4250 6700 4250 6300
-Wire Wire Line
-	4250 6300 4400 6300
-Wire Wire Line
-	4400 6300 4400 6200
-Connection ~ 4400 6300
-Wire Wire Line
-	4400 6300 4500 6300
-Wire Wire Line
-	4500 6300 4500 6400
-$Comp
-L Device:R R7
-U 1 1 5DA70518
-P 4250 6850
-F 0 "R7" V 4350 6900 50  0000 R CNN
-F 1 "10k" V 4150 6950 50  0000 R CNN
-F 2 "Resistor_SMD:R_0402_1005Metric" V 4180 6850 50  0001 C CNN
-F 3 "~" H 4250 6850 50  0001 C CNN
-F 4 "0402WGF1002TCE" H 4250 6850 50  0001 C CNN "Part Number"
-F 5 "C25744" H 4250 6850 50  0001 C CNN "LCSC Part Number"
-	1    4250 6850
-	1    0    0    -1
-$EndComp
 $Comp
 L Device:R R9
@@
 Text Label 10450 1300 0    50   ~ 0
 ZC_OUT
-NoConn ~ 10450 1900
-NoConn ~ 10450 1800
-NoConn ~ 10450 1700
 Text Label 10450 2000 0    50   ~ 0
 USR_LED
@@
 Text Notes 2150 4100 0    50   ~ 0
 Misc output
+$Comp
+L custom:LED_ARBG D13
+U 1 1 5DD14610
+P 7400 1350
+F 0 "D13" H 7400 1847 50  0000 C CNN
+F 1 "LED_ARBG" H 7400 1756 50  0000 C CNN
+F 2 "Custom:SMLP34RGB" H 7400 1300 50  0001 C CNN
+F 3 "~" H 7400 1300 50  0001 C CNN
+F 4 "SMLP34RGB2W3A" H 7400 1350 50  0001 C CNN "Part Number"
+F 5 "C162074" H 7400 1350 50  0001 C CNN "LCSC Part Number"
+	1    7400 1350
+	1    0    0    -1
+$EndComp
+$Comp
+L Device:R R38
+U 1 1 5DD5E9CF
+P 6950 1550
+F 0 "R38" V 7050 1400 50  0000 L CNN
+F 1 "47" V 7050 1600 50  0000 L CNN
+F 2 "Resistor_SMD:R_0402_1005Metric" V 6880 1550 50  0001 C CNN
+F 3 "~" H 6950 1550 50  0001 C CNN
+F 4 "0402WGF470JTCE" H 6950 1550 50  0001 C CNN "Part Number"
+F 5 "C25118" H 6950 1550 50  0001 C CNN "LCSC Part Number"
+	1    6950 1550
+	0    1    1    0
+$EndComp
+Wire Wire Line
+	7200 1150 7100 1150
+Wire Wire Line
+	7200 1350 7100 1350
+Wire Wire Line
+	7200 1550 7100 1550
+Text Label 6500 1150 2    50   ~ 0
+R_LED
+Text Label 6800 1350 2    50   ~ 0
+B_LED
+Text Label 6800 1550 2    50   ~ 0
+G_LED
+$Comp
+L power:VDD #PWR025
+U 1 1 5DDA087A
+P 7600 1350
+F 0 "#PWR025" H 7600 1200 50  0001 C CNN
+F 1 "VDD" H 7700 1450 50  0000 C CNN
+F 2 "" H 7600 1350 50  0001 C CNN
+F 3 "" H 7600 1350 50  0001 C CNN
+	1    7600 1350
+	1    0    0    -1
+$EndComp
+Text Label 10450 1700 0    50   ~ 0
+R_LED
+Text Label 10450 1800 0    50   ~ 0
+B_LED
+Text Label 10450 1900 0    50   ~ 0
+G_LED
+$Comp
+L power:VDD #PWR026
+U 1 1 5DE2586C
+P 7600 2000
+F 0 "#PWR026" H 7600 1850 50  0001 C CNN
+F 1 "VDD" H 7700 2100 50  0000 C CNN
+F 2 "" H 7600 2000 50  0001 C CNN
+F 3 "" H 7600 2000 50  0001 C CNN
+	1    7600 2000
+	1    0    0    -1
+$EndComp
+Wire Wire Line
+	7300 2000 7100 2000
+$Comp
+L Device:R R37
+U 1 1 5DE539E4
+P 6950 1350
+F 0 "R37" V 7050 1200 50  0000 L CNN
+F 1 "75" V 7050 1400 50  0000 L CNN
+F 2 "Resistor_SMD:R_0402_1005Metric" V 6880 1350 50  0001 C CNN
+F 3 "~" H 6950 1350 50  0001 C CNN
+F 4 "0402WGF750JTCE" H 6950 1350 50  0001 C CNN "Part Number"
+F 5 "C25133" H 6950 1350 50  0001 C CNN "LCSC Part Number"
+	1    6950 1350
+	0    1    1    0
+$EndComp
+$Comp
+L Device:R R7
+U 1 1 5DE55DF7
+P 6650 1150
+F 0 "R7" V 6750 1000 50  0000 L CNN
+F 1 "33" V 6750 1150 50  0000 L CNN
+F 2 "Resistor_SMD:R_0402_1005Metric" V 6580 1150 50  0001 C CNN
+F 3 "~" H 6650 1150 50  0001 C CNN
+F 4 "0402WGF330JTCE" H 6650 1150 50  0001 C CNN "Part Number"
+F 5 "C25105" H 6650 1150 50  0001 C CNN "LCSC Part Number"
+	1    6650 1150
+	0    1    1    0
+$EndComp
+$Comp
+L Device:R R36
+U 1 1 5DE53CFD
+P 6950 1150
+F 0 "R36" V 7050 1000 50  0000 L CNN
+F 1 "220" V 7050 1200 50  0000 L CNN
+F 2 "Resistor_SMD:R_0402_1005Metric" V 6880 1150 50  0001 C CNN
+F 3 "~" H 6950 1150 50  0001 C CNN
+F 4 "0402WGF2200TCE" H 6950 1150 50  0001 C CNN "Part Number"
+F 5 "C25091" H 6950 1150 50  0001 C CNN "LCSC Part Number"
+	1    6950 1150
+	0    1    1    0
+$EndComp
+$Comp
+L Device:R R8
+U 1 1 5DE5A6BC
+P 6950 2000
+F 0 "R8" V 7050 1850 50  0000 L CNN
+F 1 "220" V 7050 2000 50  0000 L CNN
+F 2 "Resistor_SMD:R_0402_1005Metric" V 6880 2000 50  0001 C CNN
+F 3 "~" H 6950 2000 50  0001 C CNN
+F 4 "0402WGF2200TCE" H 6950 2000 50  0001 C CNN "Part Number"
+F 5 "C25091" H 6950 2000 50  0001 C CNN "LCSC Part Number"
+	1    6950 2000
+	0    1    1    0
+$EndComp
 $EndSCHEMATC

Commit message: Switched USB ESD diode for STM recommened one. Added GND plane around USB traces on top layer
Parts:
- removed D8: CESD5V0AP, Package_TO_SOT_SMD:SOT-23, symbol Power_Protection:SP0502BAHT
- added C20: 100nF, Capacitor_SMD:C_0402_1005Metric, symbol Device:C
- added U5: USBLC6-2SC6, Package_TO_SOT_SMD:SOT-23-6, symbol Power_Protection:USBLC6-2SC6
Connections:
- net 5V_USB: now also C20.1, U5.5 (VBUS)
- net D+: now also R24.1, U5.6 (IO1); no longer R22.2
- net D-: now also U5.4 (IO2); no longer R23.2
- net GND: now also C20.2, U5.2 (GND)
- net USBD+: no longer R24.1
- new net: R22.2, U5.1 (IO1)
- new net: R23.2, U5.3 (IO2)
Other:
- moved on the sheet: J4, R22, R23, R24
Changed lines of the file:
@@
 L power:GND #PWR02
 U 1 1 5DE3300F
-P 5100 7000
-F 0 "#PWR02" H 5100 6750 50  0001 C CNN
-F 1 "GND" H 5105 6827 50  0000 C CNN
-F 2 "" H 5100 7000 50  0001 C CNN
-F 3 "" H 5100 7000 50  0001 C CNN
-	1    5100 7000
+P 4400 7000
+F 0 "#PWR02" H 4400 6750 50  0001 C CNN
+F 1 "GND" H 4405 6827 50  0000 C CNN
+F 2 "" H 4400 7000 50  0001 C CNN
+F 3 "" H 4400 7000 50  0001 C CNN
+	1    4400 7000
 	1    0    0    -1
 $EndComp
@@
 L power:GND #PWR01
 U 1 1 5DE3384F
-P 5000 7000
-F 0 "#PWR01" H 5000 6750 50  0001 C CNN
-F 1 "GND" H 5005 6827 50  0000 C CNN
-F 2 "" H 5000 7000 50  0001 C CNN
-F 3 "" H 5000 7000 50  0001 C CNN
-	1    5000 7000
+P 4300 7000
+F 0 "#PWR01" H 4300 6750 50  0001 C CNN
+F 1 "GND" H 4305 6827 50  0000 C CNN
+F 2 "" H 4300 7000 50  0001 C CNN
+F 3 "" H 4300 7000 50  0001 C CNN
+	1    4300 7000
 	1    0    0    -1
 $EndComp
@@
 L power:GND #PWR03
 U 1 1 5DE34D0E
-P 5400 6800
-F 0 "#PWR03" H 5400 6550 50  0001 C CNN
-F 1 "GND" H 5405 6627 50  0000 C CNN
-F 2 "" H 5400 6800 50  0001 C CNN
-F 3 "" H 5400 6800 50  0001 C CNN
-	1    5400 6800
-	1    0    0    -1
-$EndComp
-Text Label 5400 6600 0    50   ~ 0
+P 4700 6800
+F 0 "#PWR03" H 4700 6550 50  0001 C CNN
+F 1 "GND" H 4705 6627 50  0000 C CNN
+F 2 "" H 4700 6800 50  0001 C CNN
+F 3 "" H 4700 6800 50  0001 C CNN
+	1    4700 6800
+	1    0    0    -1
+$EndComp
+Text Label 4700 6600 0    50   ~ 0
 D+
-Text Label 5400 6700 0    50   ~ 0
-D-
-Text Label 4850 7400 2    50   ~ 0
-D+
-Text Label 4850 7700 2    50   ~ 0
+Text Label 4700 6700 0    50   ~ 0
 D-
 $Comp
 L Device:R R22
 U 1 1 5DE4D04E
-P 5000 7400
-F 0 "R22" V 4900 7250 50  0000 L CNN
-F 1 "22" V 4900 7450 50  0000 L CNN
-F 2 "Resistor_SMD:R_0402_1005Metric" V 4930 7400 50  0001 C CNN
-F 3 "~" H 5000 7400 50  0001 C CNN
-F 4 "0402WGF220JTCE" H 5000 7400 50  0001 C CNN "Part Number"
-F 5 "C25092" H 5000 7400 50  0001 C CNN "LCSC Part Number"
-	1    5000 7400
-	0    1    1    0
+P 4950 7350
+F 0 "R22" H 5000 7300 50  0000 L CNN
+F 1 "22" H 5000 7400 50  0000 L CNN
+F 2 "Resistor_SMD:R_0402_1005Metric" V 4880 7350 50  0001 C CNN
+F 3 "~" H 4950 7350 50  0001 C CNN
+F 4 "0402WGF220JTCE" H 4950 7350 50  0001 C CNN "Part Number"
+F 5 "C25092" H 4950 7350 50  0001 C CNN "LCSC Part Number"
+	1    4950 7350
+	-1   0    0    1
 $EndComp
 $Comp
 L Device:R R23
 U 1 1 5DE54191
-P 5000 7700
-F 0 "R23" V 4900 7550 50  0000 L CNN
-F 1 "22" V 4900 7750 50  0000 L CNN
-F 2 "Resistor_SMD:R_0402_1005Metric" V 4930 7700 50  0001 C CNN
-F 3 "~" H 5000 7700 50  0001 C CNN
-F 4 "0402WGF220JTCE" H 5000 7700 50  0001 C CNN "Part Number"
-F 5 "C25092" H 5000 7700 50  0001 C CNN "LCSC Part Number"
-	1    5000 7700
-	0    1    1    0
-$EndComp
-Text Label 5200 7650 0    50   ~ 0
-USBD-
-Text Label 5200 7350 0    50   ~ 0
-USBD+
+P 5950 7350
+F 0 "R23" H 5750 7300 50  0000 L CNN
+F 1 "22" H 5800 7400 50  0000 L CNN
+F 2 "Resistor_SMD:R_0402_1005Metric" V 5880 7350 50  0001 C CNN
+F 3 "~" H 5950 7350 50  0001 C CNN
+F 4 "0402WGF220JTCE" H 5950 7350 50  0001 C CNN "Part Number"
+F 5 "C25092" H 5950 7350 50  0001 C CNN "LCSC Part Number"
+	1    5950 7350
+	-1   0    0    1
+$EndComp
 Text Label 10450 2400 0    50   ~ 0
 USBD-
@@
 USBD+
 $Comp
-L Power_Protection:SP0502BAHT D8
-U 1 1 5DE68A64
-P 5900 7550
-F 0 "D8" V 6242 7550 50  0000 C CNN
-F 1 "CESD5V0AP" V 6151 7550 50  0000 C CNN
-F 2 "Package_TO_SOT_SMD:SOT-23" H 6125 7500 50  0001 L CNN
-F 3 "http://www.littelfuse.com/~/media/files/littelfuse/technical%20resources/documents/data%20sheets/sp05xxba.pdf" H 6025 7675 50  0001 C CNN
-F 4 "CESD5V0AP" V 5900 7550 50  0001 C CNN "Part Number"
-F 5 "" V 5900 7550 50  0001 C CNN "LCSC  Part Number"
-F 6 "C36386" H 5900 7550 50  0001 C CNN "LCSC Part Number"
-	1    5900 7550
-	0    -1   -1   0
-$EndComp
-Wire Wire Line
-	5150 7700 5200 7700
-Wire Wire Line
-	5150 7400 5200 7400
-Wire Wire Line
-	5200 7650 5200 7700
-Connection ~ 5200 7700
-Wire Wire Line
-	5200 7350 5200 7400
-Connection ~ 5200 7400
-Wire Wire Line
-	5650 7400 5650 7450
-Wire Wire Line
-	5650 7450 5700 7450
-Wire Wire Line
-	5200 7400 5650 7400
-Wire Wire Line
-	5700 7650 5650 7650
-Wire Wire Line
-	5650 7650 5650 7700
-Wire Wire Line
-	5200 7700 5650 7700
-$Comp
 L power:GND #PWR05
 U 1 1 5DEDFA16
-P 6100 7550
-F 0 "#PWR05" H 6100 7300 50  0001 C CNN
-F 1 "GND" H 6105 7377 50  0000 C CNN
-F 2 "" H 6100 7550 50  0001 C CNN
-F 3 "" H 6100 7550 50  0001 C CNN
-	1    6100 7550
+P 5450 7600
+F 0 "#PWR05" H 5450 7350 50  0001 C CNN
+F 1 "GND" H 5455 7427 50  0000 C CNN
+F 2 "" H 5450 7600 50  0001 C CNN
+F 3 "" H 5450 7600 50  0001 C CNN
+	1    5450 7600
 	1    0    0    -1
 $EndComp
@@
 L Device:R R24
 U 1 1 5DF21CB4
-P 5850 6750
-F 0 "R24" H 5900 6750 50  0000 L CNN
-F 1 "2k" H 5900 6850 50  0000 L CNN
-F 2 "Resistor_SMD:R_0402_1005Metric" V 5780 6750 50  0001 C CNN
-F 3 "~" H 5850 6750 50  0001 C CNN
-F 4 "0402WGF2001TCE" H 5850 6750 50  0001 C CNN "Part Number"
-F 5 "C4109" H 5850 6750 50  0001 C CNN "LCSC Part Number"
-	1    5850 6750
+P 5900 6350
+F 0 "R24" H 5950 6350 50  0000 L CNN
+F 1 "2k" H 5950 6450 50  0000 L CNN
+F 2 "Resistor_SMD:R_0402_1005Metric" V 5830 6350 50  0001 C CNN
+F 3 "~" H 5900 6350 50  0001 C CNN
+F 4 "0402WGF2001TCE" H 5900 6350 50  0001 C CNN "Part Number"
+F 5 "C4109" H 5900 6350 50  0001 C CNN "LCSC Part Number"
+	1    5900 6350
 	-1   0    0    1
 $EndComp
@@
 L Connector:USB_B_Micro J4
 U 1 1 5DE25992
-P 5100 6600
-F 0 "J4" H 5100 7050 50  0000 C CNN
-F 1 "USB_B_Micro" H 5150 6950 50  0000 C CNN
-F 2 "Custom:ZX62M-B-5P(30)" H 5250 6550 50  0001 C CNN
-F 3 "~" H 5250 6550 50  0001 C CNN
-	1    5100 6600
-	1    0    0    -1
-$EndComp
-Text Label 5400 6400 0    50   ~ 0
+P 4400 6600
+F 0 "J4" H 4400 7050 50  0000 C CNN
+F 1 "USB_B_Micro" H 4450 6950 50  0000 C CNN
+F 2 "Custom:ZX62M-B-5P(30)" H 4550 6550 50  0001 C CNN
+F 3 "~" H 4550 6550 50  0001 C CNN
+	1    4400 6600
+	1    0    0    -1
+$EndComp
+Text Label 4700 6400 0    50   ~ 0
 5V_USB
-Text Label 5850 6950 0    50   ~ 0
-USBD+
-Wire Wire Line
-	5850 6950 5850 6900
+Wire Wire Line
+	5900 6550 5900 6500
 Text Label 2800 5450 2    50   ~ 0
 5V_MAINS
@@
 Wire Notes Line
 	3650 6100 3650 7750
-Wire Notes Line
-	4700 6100 4700 7750
-Text Notes 4800 6200 0    50   ~ 0
+Text Notes 4150 6200 0    50   ~ 0
 USB
 Text Notes 6250 6600 0    50   ~ 0
@@
 	-1   0    0    1
 $EndComp
-Text Label 5850 6600 0    50   ~ 0
+Text Label 5900 6200 0    50   ~ 0
 5V_USB
 Wire Notes Line
@@
 	0    1    1    0
 $EndComp
+Text Label 5900 6550 0    50   ~ 0
+D+
+$Comp
+L Power_Protection:USBLC6-2SC6 U5
+U 1 1 5E02C90F
+P 5450 7100
+F 0 "U5" H 5200 7450 50  0000 C CNN
+F 1 "USBLC6-2SC6" H 5800 7450 50  0000 C CNN
+F 2 "Package_TO_SOT_SMD:SOT-23-6" H 4700 7500 50  0001 C CNN
+F 3 "http://www2.st.com/resource/en/datasheet/CD00050750.pdf" H 5650 7450 50  0001 C CNN
+F 4 "C7519" H 5450 7100 50  0001 C CNN "LCSC Part Number"
+F 5 "USBLC6-2SC6" H 5450 7100 50  0001 C CNN "Part Number"
+	1    5450 7100
+	1    0    0    -1
+$EndComp
+Text Label 4950 7000 2    50   ~ 0
+D+
+Text Label 4950 7500 0    50   ~ 0
+USBD+
+Text Label 5950 7000 0    50   ~ 0
+D-
+Text Label 5950 7500 2    50   ~ 0
+USBD-
+Text Label 5450 6600 0    50   ~ 0
+5V_USB
+$Comp
+L Device:C C20
+U 1 1 5E08E89F
+P 5150 6350
+F 0 "C20" H 5150 6450 50  0000 L CNN
+F 1 "100nF" H 5150 6250 50  0000 L CNN
+F 2 "Capacitor_SMD:C_0402_1005Metric" H 5188 6200 50  0001 C CNN
+F 3 "~" H 5150 6350 50  0001 C CNN
+F 4 "CL05B104KO5NNNC" H 5150 6350 50  0001 C CNN "Part Number"
+F 5 "C1525" H 5150 6350 50  0001 C CNN "LCSC Part Number"
+	1    5150 6350
+	1    0    0    -1
+$EndComp
+Wire Notes Line
+	4700 7250 4700 7750
+Text Label 5150 6200 0    50   ~ 0
+5V_USB
+$Comp
+L power:GND #PWR027
+U 1 1 5E15DD07
+P 5150 6500
+F 0 "#PWR027" H 5150 6250 50  0001 C CNN
+F 1 "GND" H 5155 6327 50  0000 C CNN
+F 2 "" H 5150 6500 50  0001 C CNN
+F 3 "" H 5150 6500 50  0001 C CNN
+	1    5150 6500
+	1    0    0    -1
+$EndComp
 $EndSCHEMATC

Commit message: Added hw debouncing to trigger. Added SCL pull-up. Made both I2C pull-ups 2.2k and optional
Parts:
- added C23: 10nf, Capacitor_SMD:C_0402_1005Metric, symbol Device:C
- added JP1, JP2: SolderJumper_2_Open, Jumper:SolderJumper-2_P1.3mm_Open_TrianglePad1.0x1.5mm, symbol Jumper:SolderJumper_2_Open
- added R39: 10k, Resistor_SMD:R_0402_1005Metric, symbol Device:R
- added R40: 2.2k, Resistor_SMD:R_0402_1005Metric, symbol Device:R
- R19: value 4.7k -> 2.2k; LCSC Part Number C25900 -> C25879; Part Number 0402WGF4701TCE -> 0402WGF2201TCE
Connections:
- net GND: now also C23.2
- net SCL: now also R40.2
- net Trigger: now also C23.1, R39.1; no longer J3.17 (Pin_17), R14.1
- net VCC: now also JP1.1 (A), JP2.1 (A); no longer R19.1
- new net: JP2.2 (B), R19.1
- new net: JP1.2 (B), R40.1
- new net Trigger_RAW: J3.17 (Pin_17), R14.1, R39.2
Other:
- moved on the sheet: D10, D11, R14, R18

Commit message: Shuffled board around to put AC/DC right on the edge so hopefully it will fit alongside an SSR mounted in the lid of the box
Parts:
- JP1, JP2: footprint Jumper:SolderJumper-2_P1.3mm_Open_TrianglePad1.0x1.5mm -> Custom:SolderJumper-2_P1.3mm_Open_TrianglePad1.0x1.5mm
Changed lines of the file:
@@
 F 0 "JP2" V 2300 6500 50  0000 L CNN
 F 1 "SolderJumper_2_Open" V 2450 6450 50  0001 L CNN
-F 2 "Jumper:SolderJumper-2_P1.3mm_Open_TrianglePad1.0x1.5mm" H 2350 6650 50  0001 C CNN
+F 2 "Custom:SolderJumper-2_P1.3mm_Open_TrianglePad1.0x1.5mm" H 2350 6650 50  0001 C CNN
 F 3 "~" H 2350 6650 50  0001 C CNN
 	1    2350 6650
@@
 F 0 "JP1" V 2300 5650 50  0000 L CNN
 F 1 "SolderJumper_2_Open" V 2450 5600 50  0001 L CNN
-F 2 "Jumper:SolderJumper-2_P1.3mm_Open_TrianglePad1.0x1.5mm" H 2350 5800 50  0001 C CNN
+F 2 "Custom:SolderJumper-2_P1.3mm_Open_TrianglePad1.0x1.5mm" H 2350 5800 50  0001 C CNN
 F 3 "~" H 2350 5800 50  0001 C CNN
 	1    2350 5800
