File: hardware/zero_crossing_detector_surface_mount/zero_crossing_detector.sch (KiCad schematic (older format))
At the start: 98 parts, among them J1 Conn_01x02, J2 BOOT0, J3 Conn_02x15_Odd_Even, J4 USB_B_Micro, J6 K-Type, J7 BOOT1, Q1 2N3904, Q2 2N3904, Q3 2N3904, SW1 Reset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

Commit message: Removed RGB led
Parts:
- removed D13: LED_ARBG, Custom:SMLP34RGB, symbol custom:LED_ARBG
- removed R36: 220, Resistor_SMD:R_0402_1005Metric, symbol Device:R
- removed R37: 75, Resistor_SMD:R_0402_1005Metric, symbol Device:R
- removed R38: 47, Resistor_SMD:R_0402_1005Metric, symbol Device:R
- removed R7: 33, Resistor_SMD:R_0402_1005Metric, symbol Device:R
Connections:
- net B_LED: no longer names the net of U2.21 (PA5)
- net G_LED: no longer names the net of U2.22 (PA6)
- net R_LED: no longer names the net of U2.20 (PA4)
- no-connect marks 23 -> 26
Changed lines of the file:
@@
 Misc output
-$Comp
-L custom:LED_ARBG D13
-U 1 1 5DD14610
-P 7400 1350
-F 0 "D13" H 7400 1847 50  0000 C CNN
-F 1 "LED_ARBG" H 7400 1756 50  0000 C CNN
-F 2 "Custom:SMLP34RGB" H 7400 1300 50  0001 C CNN
-F 3 "~" H 7400 1300 50  0001 C CNN
-F 4 "SMLP34RGB2W3A" H 7400 1350 50  0001 C CNN "Part Number"
-F 5 "C162074" H 7400 1350 50  0001 C CNN "LCSC Part Number"
-	1    7400 1350
-	1    0    0    -1
-$EndComp
-$Comp
-L Device:R R38
-U 1 1 5DD5E9CF
-P 6950 1550
-F 0 "R38" V 7050 1400 50  0000 L CNN
-F 1 "47" V 7050 1600 50  0000 L CNN
-F 2 "Resistor_SMD:R_0402_1005Metric" V 6880 1550 50  0001 C CNN
-F 3 "~" H 6950 1550 50  0001 C CNN
-F 4 "0402WGF470JTCE" H 6950 1550 50  0001 C CNN "Part Number"
-F 5 "C25118" H 6950 1550 50  0001 C CNN "LCSC Part Number"
-	1    6950 1550
-	0    1    1    0
-$EndComp
-Wire Wire Line
-	7200 1150 7100 1150
-Wire Wire Line
-	7200 1350 7100 1350
-Wire Wire Line
-	7200 1550 7100 1550
-Text Label 6500 1150 2    50   ~ 0
-R_LED
-Text Label 6800 1350 2    50   ~ 0
-B_LED
-Text Label 6800 1550 2    50   ~ 0
-G_LED
-$Comp
-L power:VDD #PWR025
-U 1 1 5DDA087A
-P 7600 1350
-F 0 "#PWR025" H 7600 1200 50  0001 C CNN
-F 1 "VDD" H 7700 1450 50  0000 C CNN
-F 2 "" H 7600 1350 50  0001 C CNN
-F 3 "" H 7600 1350 50  0001 C CNN
-	1    7600 1350
-	1    0    0    -1
-$EndComp
-Text Label 10450 1700 0    50   ~ 0
-R_LED
-Text Label 10450 1800 0    50   ~ 0
-B_LED
-Text Label 10450 1900 0    50   ~ 0
-G_LED
 $Comp
 L power:VDD #PWR026
@@
 Wire Wire Line
 	7300 2000 7100 2000
-$Comp
-L Device:R R37
-U 1 1 5DE539E4
-P 6950 1350
-F 0 "R37" V 7050 1200 50  0000 L CNN
-F 1 "75" V 7050 1400 50  0000 L CNN
-F 2 "Resistor_SMD:R_0402_1005Metric" V 6880 1350 50  0001 C CNN
-F 3 "~" H 6950 1350 50  0001 C CNN
-F 4 "0402WGF750JTCE" H 6950 1350 50  0001 C CNN "Part Number"
-F 5 "C25133" H 6950 1350 50  0001 C CNN "LCSC Part Number"
-	1    6950 1350
-	0    1    1    0
-$EndComp
-$Comp
-L Device:R R7
-U 1 1 5DE55DF7
-P 6650 1150
-F 0 "R7" V 6750 1000 50  0000 L CNN
-F 1 "33" V 6750 1150 50  0000 L CNN
-F 2 "Resistor_SMD:R_0402_1005Metric" V 6580 1150 50  0001 C CNN
-F 3 "~" H 6650 1150 50  0001 C CNN
-F 4 "0402WGF330JTCE" H 6650 1150 50  0001 C CNN "Part Number"
-F 5 "C25105" H 6650 1150 50  0001 C CNN "LCSC Part Number"
-	1    6650 1150
-	0    1    1    0
-$EndComp
-$Comp
-L Device:R R36
-U 1 1 5DE53CFD
-P 6950 1150
-F 0 "R36" V 7050 1000 50  0000 L CNN
-F 1 "220" V 7050 1200 50  0000 L CNN
-F 2 "Resistor_SMD:R_0402_1005Metric" V 6880 1150 50  0001 C CNN
-F 3 "~" H 6950 1150 50  0001 C CNN
-F 4 "0402WGF2200TCE" H 6950 1150 50  0001 C CNN "Part Number"
-F 5 "C25091" H 6950 1150 50  0001 C CNN "LCSC Part Number"
-	1    6950 1150
-	0    1    1    0
-$EndComp
 $Comp
 L Device:R R8
@@
 	0    1    1    0
 $EndComp
+NoConn ~ 10450 1700
+NoConn ~ 10450 1800
+NoConn ~ 10450 1900
 $EndSCHEMATC
